Commit message: Go 4 wheel. Tweak dependencies (gazebo_ros is gazebo classic).

File: model/robot.xacro (robot description, xacro)
@@ -1,4 +1,4 @@
 <?xml version="1.0"?>
-<robot name="differential_drive_robot" xmlns:xacro="http://www.ros.org/wiki/xacro">
+<robot name="differential_drive_robot_4wheel" xmlns:xacro="http://www.ros.org/wiki/xacro">
     <!-- Robot Parameters -->
     <xacro:property name="PI" value="3.14159265"/>
@@ -12,5 +12,5 @@
     <xacro:property name="body_inertia_z" value="${1.0/12.0 * body_mass * (body_length*body_length + body_width*body_width)}"/>
     <xacro:property name="wheel_radius" value="0.1"/>
-    <xacro:property name="wheel_width" value="0.05"/>
+    <xacro:property name="wheel_width" value="0.1"/>
     <xacro:property name="wheel_separation" value="${body_width + wheel_width}"/>
     <xacro:property name="wheel_offset" value="${body_length/2 - wheel_radius}"/>
@@ -99,6 +99,52 @@
         </inertial>
     </link>
+    <!-- Left Wheel 2 -->
+    <link name="left_wheel2_link">
+        <visual>
+            <origin xyz="0.0 0.0 0.0" rpy="1.570795 0.0 0.0"/>
+            <geometry>
+                <cylinder radius="${wheel_radius}" length="${wheel_width}"/>
+            </geometry>
+            <material name="wheel_material">
+                <color rgba="0.0 0.0 0.0 1.0"/>
+            </material>
+        </visual>
+        <collision>
+            <origin xyz="0.0 0.0 0.0" rpy="1.570795 0.0 0.0"/>
+            <geometry>
+                <cylinder radius="${wheel_radius}" length="${wheel_width}"/>
+            </geometry>
+        </collision>
+        <inertial>
+            <mass value="2"/>
+            <inertia ixx="${wheel_inertia_x}" ixy="0.0" ixz="0.0" iyy="${wheel_inertia_y}" iyz="0" izz="${wheel_inertia_z}"/>
+            <origin xyz="0.0 0.0 0.0" rpy="1.570795 0.0 0.0"/>
+        </inertial>
+    </link>
+    <!-- Right Wheel 2-->
+    <link name="right_wheel2_link">
+        <visual>
+            <origin xyz="0.0 0.0 0.0" rpy="1.570795 0.0 0.0"/>
+            <geometry>
+                <cylinder radius="${wheel_radius}" length="${wheel_width}"/>
+            </geometry>
+            <material name="wheel_material">
+                <color rgba="0.0 0.0 0.0 1.0"/>
+            </material>
+        </visual>
+        <collision>
+            <origin xyz="0.0 0.0 0.0" rpy="1.570795 0.0 0.0"/>
+            <geometry>
+                <cylinder radius="${wheel_radius}" length="${wheel_width}"/>
+            </geometry>
+        </collision>
+        <inertial>
+            <mass value="2"/>
+            <inertia ixx="${wheel_inertia_x}" ixy="0.0" ixz="0.0" iyy="${wheel_inertia_y}" iyz="0" izz="${wheel_inertia_z}"/>
+            <origin xyz="0.0 0.0 0.0" rpy="1.570795 0.0 0.0"/>
+        </inertial>
+    </link>
     <!-- Caster Wheel -->
-    <link name="caster_link">
+<!--    <link name="caster_link">
         <visual>
             <origin xyz="0.0 0.0 0.0" rpy="0.0 0.0 0.0"/>
@@ -121,5 +167,5 @@
             <origin xyz="0 0 0" rpy="0 0 0"/>
         </inertial>
-    </link>
+    </link>-->
     <!-- Joints -->
     <!-- Left Wheel Joint -->
@@ -141,10 +187,28 @@
         <dynamics damping="0.1" friction="0.1"/>
     </joint>
+    <!-- Left Wheel2 Joint -->
+    <joint name="left_wheel2_joint" type="continuous">
+        <origin xyz="${wheel_offset} ${wheel_separation/2} -${wheel_radius/2}" rpy="0 0 0"/>
+        <parent link="body_link"/>
+        <child link="left_wheel2_link"/>
+        <axis xyz="0 1 0"/>
+        <limit effort="100" velocity="10.0"/>
+        <dynamics damping="0.1" friction="0.1"/>
+    </joint>
+    <!-- Right Wheel2 Joint -->
+    <joint name="right_wheel2_joint" type="continuous">
+        <origin xyz="${wheel_offset} ${-wheel_separation/2} -${wheel_radius/2}" rpy="0 0 0"/>
+        <parent link="body_link"/>
+        <child link="right_wheel2_link"/>
+        <axis xyz="0 1 0"/>
+        <limit effort="100" velocity="10.0"/>
+        <dynamics damping="0.1" friction="0.1"/>
+    </joint>
     <!-- Caster Wheel Joint (fixed) -->
-    <joint name="caster_joint" type="fixed">
+<!--    <joint name="caster_joint" type="fixed">
         <origin xyz="${caster_offset} 0 -${caster_radius/2}" rpy="0 0 0"/>
         <parent link="body_link"/>
         <child link="caster_link"/>
-    </joint>
+    </joint>-->
     <!-- Gazebo Parameters -->
     <gazebo reference="body_link">
@@ -160,8 +224,16 @@
         <mu2>1.0</mu2>
     </gazebo>
-    <gazebo reference="caster_link">
+    <gazebo reference="right_wheel2_link">
+        <mu1>1.0</mu1>
+        <mu2>1.0</mu2>
+    </gazebo>
+    <gazebo reference="left_wheel2_link">
+        <mu1>1.0</mu1>
+        <mu2>1.0</mu2>
+    </gazebo>
+<!--    <gazebo reference="caster_link">
         <mu1>0.000001</mu1>
         <mu2>0.000001</mu2>
-    </gazebo>
+    </gazebo>-->
     <!-- Gazebo Plugins -->
     <gazebo>
@@ -169,4 +241,6 @@
             <right_joint>right_wheel_joint</right_joint>
             <left_joint>left_wheel_joint</left_joint>
+            <right_joint>right_wheel2_joint</right_joint>
+            <left_joint>left_wheel2_joint</left_joint>
             <wheel_separation>${wheel_separation}</wheel_separation>
             <wheel_radius>${wheel_radius}</wheel_radius>
@@ -180,4 +254,6 @@
             <joint_name>right_wheel_joint</joint_name>
             <joint_name>left_wheel_joint</joint_name>
+            <joint_name>right_wheel2_joint</joint_name>
+            <joint_name>left_wheel2_joint</joint_name>
         </plugin>
     </gazebo>
