Commit message: Update xacro for a reasonable facsimile of the entire robot - sans sensors (this is next).

File: model/robot.xacro (robot description, xacro)
@@ -1,175 +1,133 @@
 <?xml version="1.0"?>
 <robot name="differential_drive_robot_4wheel" xmlns:xacro="http://www.ros.org/wiki/xacro">
+    <xacro:macro name="box_link" params="name length width height density color">
+        <!-- Compute mass -->
+        <xacro:property name="volume" value="${length * width * height}"/>
+        <xacro:property name="mass" value="${density * volume}"/>
+        <!-- Inertia for a box centered at origin -->
+        <xacro:property name="ixx" value="${(1.0/12.0) * mass * (height**2 + width**2)}"/>
+        <xacro:property name="iyy" value="${(1.0/12.0) * mass * (length**2 + height**2)}"/>
+        <xacro:property name="izz" value="${(1.0/12.0) * mass * (length**2 + width**2)}"/>
+        <link name="${name}">
+          <visual>
+            <origin xyz="0 0 0" rpy="0 0 0"/>
+            <geometry>
+              <box size="${length} ${width} ${height}"/>
+            </geometry>
+            <material name="${name}_material">
+              <color rgba="${color}"/>
+            </material>
+          </visual>
+          <collision>
+            <origin xyz="0 0 0" rpy="0 0 0"/>
+            <geometry>
+              <box size="${length} ${width} ${height}"/>
+            </geometry>
+          </collision>
+          <inertial>
+            <origin xyz="0 0 0" rpy="0 0 0"/>
+            <mass value="${mass}"/>
+            <inertia
+              ixx="${ixx}" ixy="0.0" ixz="0.0"
+              iyy="${iyy}" iyz="0.0"
+              izz="${izz}"/>
+          </inertial>
+        </link>
+    </xacro:macro>
+    <xacro:macro name="wheel_link" params="name radius width density color">
+        <!-- Volume and mass -->
+        <xacro:property name="volume" value="${pi * radius**2 * width}"/>
+        <xacro:property name="mass" value="${density * volume}"/>
+        <!-- Solid cylinder inertias (rotated about its own Z axis) -->
+        <!-- Assume rotation axis (wheel spin) is along the X axis (due to roll of π/2) -->
+        <xacro:property name="ixx" value="${0.5 * mass * radius**2}"/> <!-- spin axis -->
+        <xacro:property name="iyy" value="${0.25 * mass * radius**2 + (1.0/12.0) * mass * width**2}"/>
+        <xacro:property name="izz" value="${iyy}"/>
+        <link name="${name}">
+          <visual>
+            <origin xyz="0 0 0" rpy="${pi/2} 0 0"/> <!-- roll = pi/2 -->
+            <geometry>
+              <cylinder radius="${radius}" length="${width}"/>
+            </geometry>
+            <material name="${name}_material">
+              <color rgba="${color}"/>
+            </material>
+          </visual>
+          <collision>
+            <origin xyz="0 0 0" rpy="${pi/2} 0 0"/> <!-- roll = pi/2 -->
+            <geometry>
+              <cylinder radius="${radius}" length="${width}"/>
+            </geometry>
+          </collision>
+          <inertial>
+            <origin xyz="0 0 0" rpy="0 0 0"/>
+            <mass value="${mass}"/>
+            <inertia
+              ixx="${ixx}" ixy="0.0" ixz="0.0"
+              iyy="${iyy}" iyz="0.0"
+              izz="${izz}"/>
+          </inertial>
+        </link>
+    </xacro:macro>
     <!-- Robot Parameters -->
-    <xacro:property name="PI" value="3.14159265"/>
-    <xacro:property name="body_length" value="0.5"/>
-    <xacro:property name="body_width" value="0.3"/>
-    <xacro:property name="body_height" value="0.1"/>
-    <xacro:property name="body_density" value="7850.0"/> <!-- Steel -->
-    <xacro:property name="body_mass" value="${body_density * body_length * body_height * body_width}"/>
-    <xacro:property name="body_inertia_x" value="${1.0/12.0 * body_mass * (body_height*body_height + body_width*body_width)}"/>
-    <xacro:property name="body_inertia_y" value="${1.0/12.0 * body_mass * (body_length*body_length + body_height*body_height)}"/>
-    <xacro:property name="body_inertia_z" value="${1.0/12.0 * body_mass * (body_length*body_length + body_width*body_width)}"/>
-    <xacro:property name="wheel_radius" value="0.1"/>
-    <xacro:property name="wheel_width" value="0.1"/>
-    <xacro:property name="wheel_separation" value="${body_width + wheel_width}"/>
+    <xacro:property name="velcro_height" value=".006"/>
+    <xacro:property name="body_length" value="0.24"/>
+    <xacro:property name="body_width" value="0.120"/>
+    <xacro:property name="body_height" value="0.06"/>
+    <xacro:property name="body_ground_clearance" value="0.021"/>
+    <xacro:property name="body_density" value="2700.0"/> <!-- Aluminum -->
+    <xacro:property name="wheel_radius" value="0.039"/>
+    <xacro:property name="wheel_width" value="0.042"/>
+    <xacro:property name="body_wheel_gap" value="0.006"/>
+    <xacro:property name="body_wheel_axle_offset" value="${(wheel_radius-body_ground_clearance) - body_height/2.0}"/>
+    <xacro:property name="wheel_separation" value="${body_width + wheel_width + 2*body_wheel_gap}"/>
     <xacro:property name="wheel_offset" value="${body_length/2 - wheel_radius}"/>
-    <xacro:property name="wheel_density" value="900"/> <!-- Ruber -->
-    <xacro:property name="wheel_mass" value="${wheel_density * PI * wheel_radius * wheel_radius * wheel_width}"/>
-    <xacro:property name="wheel_inertia_x" value="${1.0/12.0 * wheel_mass * (3*wheel_radius*wheel_radius + wheel_width*wheel_width)}"/>
-    <xacro:property name="wheel_inertia_y" value="${1.0/12.0 * wheel_mass * (3*wheel_radius*wheel_radius + wheel_width*wheel_width)}"/>
-    <xacro:property name="wheel_inertia_z" value="${1.0/2.0 * wheel_mass * wheel_radius * wheel_radius}"/>
-    <xacro:property name="caster_radius" value="0.1"/>
-    <xacro:property name="caster_offset" value="${body_length/2 - caster_radius}"/>
-    <xacro:property name="caster_density" value="0.1"/>
-    <xacro:property name="caster_mass" value="${caster_density * 4.0/3.0 * PI * caster_radius * caster_radius * caster_radius}"/>
-    <xacro:property name="caster_inertia_x" value="${2.0/5.0 * caster_mass * caster_radius * caster_radius}"/>
-    <xacro:property name="caster_inertia_y" value="${2.0/5.0 * caster_mass * caster_radius * caster_radius}"/>
-    <xacro:property name="caster_inertia_z" value="${2.0/5.0 * caster_mass * caster_radius * caster_radius}"/>
+    <xacro:property name="wheel_density" value="900"/> <!-- Rubber -->
+    <xacro:property name="orin_length" value="0.110"/>
+    <xacro:property name="orin_width" value="0.110"/>
+    <xacro:property name="orin_height" value="0.072"/>
+    <xacro:property name="orin_density" value="2700.0"/> <!-- Aluminum -->
+    <xacro:property name="battery_length" value="0.095"/>
+    <xacro:property name="battery_width" value="0.190"/>
+    <xacro:property name="battery_height" value="0.027"/>
+    <xacro:property name="battery_density" value="2700.0"/> <!-- aluminum -->
+    <xacro:property name="lidar_length" value="0.038"/>
+    <xacro:property name="lidar_width" value="0.038"/>
+    <xacro:property name="lidar_height" value="0.035"/>
+    <xacro:property name="lidar_density" value="900.0"/> <!-- plastic-->
+    <xacro:property name="d435_length" value="0.024"/>
+    <xacro:property name="d435_width" value="0.090"/>
+    <xacro:property name="d435_height" value="0.025"/>
+    <xacro:property name="d435_density" value="900.0"/> <!-- plastic-->
+    <xacro:property name="gps_length" value="0.025"/>
+    <xacro:property name="gps_width" value="0.042"/>
+    <xacro:property name="gps_height" value="0.008"/>
+    <xacro:property name="gps_density" value="900.0"/> <!-- plastic-->
+    <xacro:property name="body_battery_offset" value="${body_height/2 + battery_height/2 + velcro_height}"/>
+    <xacro:property name="battery_orin_offset" value="${battery_height/2 + orin_height/2 + velcro_height}"/>
+    <xacro:property name="orin_lidar_offset" value="${orin_height/2 + lidar_height/2 + velcro_height}"/>
+    <xacro:property name="orin_d435_offset_x" value="${orin_length/2 + d435_length/2 + velcro_height}"/>
+    <xacro:property name="orin_d435_offset_z" value="${orin_height/2 - d435_height/2}"/>
+    <xacro:property name="orin_gps_offset_x" value=".034"/>
+    <xacro:property name="orin_gps_offset_y" value="-${orin_width/2 + gps_width/2}"/>
+    <xacro:property name="orin_gps_offset_z" value="-${orin_height/2 - .020}"/>
     <!-- Control Parameters -->
     <xacro:property name="max_linear_acceleration" value="10"/>
     <!-- Links -->
     <!-- Body Link -->
-    <link name="body_link">
-        <visual>
-            <origin xyz="0.0 0.0 0.0" rpy="0.0 0.0 0.0"/>
-            <geometry>
-                <box size="${body_length} ${body_width} ${body_height}"/>
-            </geometry>
-            <material name="body_material">
-                <color rgba="0.25 0.25 0.25 1.0"/>
-            </material>
-        </visual>
-        <collision>
-            <origin xyz="0.0 0.0 0.0" rpy="0.0 0.0 0.0"/>
-            <geometry>
-                <box size="${body_length} ${body_width} ${body_height}"/>
-            </geometry>
-        </collision>
-        <inertial>
-            <mass value="10"/>
-            <inertia ixx="${body_inertia_x}" ixy="0.0" ixz="0.0" iyy="${body_inertia_y}" iyz="0" izz="${body_inertia_z}"/>
-            <origin xyz="0 0 0" rpy="0 0 0"/>
-        </inertial>
-    </link>
-    <!-- Left Wheel -->
-    <link name="left_wheel_link">
-        <visual>
-            <origin xyz="0.0 0.0 0.0" rpy="1.570795 0.0 0.0"/>
-            <geometry>
-                <cylinder radius="${wheel_radius}" length="${wheel_width}"/>
-            </geometry>
-            <material name="wheel_material">
-                <color rgba="0.0 0.0 0.0 1.0"/>
-            </material>
-        </visual>
-        <collision>
-            <origin xyz="0.0 0.0 0.0" rpy="1.570795 0.0 0.0"/>
-            <geometry>
-                <cylinder radius="${wheel_radius}" length="${wheel_width}"/>
-            </geometry>
-        </collision>
-        <inertial>
-            <mass value="2"/>
-            <inertia ixx="${wheel_inertia_x}" ixy="0.0" ixz="0.0" iyy="${wheel_inertia_y}" iyz="0" izz="${wheel_inertia_z}"/>
-            <origin xyz="0.0 0.0 0.0" rpy="1.570795 0.0 0.0"/>
-        </inertial>
-    </link>
-    <!-- Right Wheel -->
-    <link name="right_wheel_link">
-        <visual>
-            <origin xyz="0.0 0.0 0.0" rpy="1.570795 0.0 0.0"/>
-            <geometry>
-                <cylinder radius="${wheel_radius}" length="${wheel_width}"/>
-            </geometry>
-            <material name="wheel_material">
-                <color rgba="0.0 0.0 0.0 1.0"/>
-            </material>
-        </visual>
-        <collision>
-            <origin xyz="0.0 0.0 0.0" rpy="1.570795 0.0 0.0"/>
-            <geometry>
-                <cylinder radius="${wheel_radius}" length="${wheel_width}"/>
-            </geometry>
-        </collision>
-        <inertial>
-            <mass value="2"/>
-            <inertia ixx="${wheel_inertia_x}" ixy="0.0" ixz="0.0" iyy="${wheel_inertia_y}" iyz="0" izz="${wheel_inertia_z}"/>
-            <origin xyz="0.0 0.0 0.0" rpy="1.570795 0.0 0.0"/>
-        </inertial>
-    </link>
-    <!-- Left Wheel 2 -->
-    <link name="left_wheel2_link">
-        <visual>
-            <origin xyz="0.0 0.0 0.0" rpy="1.570795 0.0 0.0"/>
-            <geometry>
-                <cylinder radius="${wheel_radius}" length="${wheel_width}"/>
-            </geometry>
-            <material name="wheel_material">
-                <color rgba="0.0 0.0 0.0 1.0"/>
-            </material>
-        </visual>
-        <collision>
-            <origin xyz="0.0 0.0 0.0" rpy="1.570795 0.0 0.0"/>
-            <geometry>
-                <cylinder radius="${wheel_radius}" length="${wheel_width}"/>
-            </geometry>
-        </collision>
-        <inertial>
-            <mass value="2"/>
-            <inertia ixx="${wheel_inertia_x}" ixy="0.0" ixz="0.0" iyy="${wheel_inertia_y}" iyz="0" izz="${wheel_inertia_z}"/>
-            <origin xyz="0.0 0.0 0.0" rpy="1.570795 0.0 0.0"/>
-        </inertial>
-    </link>
-    <!-- Right Wheel 2-->
-    <link name="right_wheel2_link">
-        <visual>
-            <origin xyz="0.0 0.0 0.0" rpy="1.570795 0.0 0.0"/>
-            <geometry>
-                <cylinder radius="${wheel_radius}" length="${wheel_width}"/>
-            </geometry>
-            <material name="wheel_material">
-                <color rgba="0.0 0.0 0.0 1.0"/>
-            </material>
-        </visual>
-        <collision>
-            <origin xyz="0.0 0.0 0.0" rpy="1.570795 0.0 0.0"/>
-            <geometry>
-                <cylinder radius="${wheel_radius}" length="${wheel_width}"/>
-            </geometry>
-        </collision>
-        <inertial>
-            <mass value="2"/>
-            <inertia ixx="${wheel_inertia_x}" ixy="0.0" ixz="0.0" iyy="${wheel_inertia_y}" iyz="0" izz="${wheel_inertia_z}"/>
-            <origin xyz="0.0 0.0 0.0" rpy="1.570795 0.0 0.0"/>
-        </inertial>
-    </link>
-    <!-- Caster Wheel -->
-<!--    <link name="caster_link">
-        <visual>
-            <origin xyz="0.0 0.0 0.0" rpy="0.0 0.0 0.0"/>
-            <geometry>
-                <sphere radius="${caster_radius}"/>
-            </geometry>
-            <material name="caster_material">
-                <color rgba="0.0 0.0 0.0 1.0"/>
-            </material>
-        </visual>
-        <collision>
-            <origin xyz="0.0 0.0 0.0" rpy="0.0 0.0 0.0"/>
-            <geometry>
-                <sphere radius="${caster_radius}"/>
-            </geometry>
-        </collision>
-        <inertial>
-            <mass value="0.5"/>
-            <inertia ixx="${caster_inertia_x}" ixy="0.0" ixz="0.0" iyy="${caster_inertia_y}" iyz="0" izz="${caster_inertia_z}"/>
-            <origin xyz="0 0 0" rpy="0 0 0"/>
-        </inertial>
-    </link>-->
+    <xacro:box_link name="body_link" length="${body_length}" width="${body_width}" height="${body_height}" density="${body_density}" color="0.0 0.0 0.0 1.0"/>
+    <xacro:box_link name="battery_link" length="${battery_length}" width="${battery_width}" height="${battery_height}" density="${battery_density}" color="0.25 0.25 0.25 1.0"/>
+    <xacro:box_link name="orin_link" length="${orin_length}" width="${orin_width}" height="${orin_height}" density="${orin_density}" color="0.45 0.45 0.45 1.0"/>
+    <xacro:box_link name="lidar_link" length="${lidar_length}" width="${lidar_width}" height="${lidar_height}" density="${lidar_density}" color="0.0 0.0 0.0 1.0"/>
+    <xacro:box_link name="d435_link" length="${d435_length}" width="${d435_width}" height="${d435_height}" density="${d435_density}" color="0.7 0.7 0.7 1.0"/>
+    <xacro:box_link name="gps_link" length="${gps_length}" width="${gps_width}" height="${gps_height}" density="${gps_density}" color="1.0 1.0 1.0 1.0"/>
+    <xacro:wheel_link name="left_wheel_link" radius="${wheel_radius}" width="${wheel_width}" density="${wheel_density}" color="0.1 0.1 0.1 1.0"/>
+    <xacro:wheel_link name="right_wheel_link" radius="${wheel_radius}" width="${wheel_width}" density="${wheel_density}" color="0.1 0.1 0.1 1.0"/>
+    <xacro:wheel_link name="left_wheel2_link" radius="${wheel_radius}" width="${wheel_width}" density="${wheel_density}" color="0.1 0.1 0.1 1.0"/>
+    <xacro:wheel_link name="right_wheel2_link" radius="${wheel_radius}" width="${wheel_width}" density="${wheel_density}" color="0.1 0.1 0.1 1.0"/>
     <!-- Joints -->
     <!-- Left Wheel Joint -->
     <joint name="left_wheel_joint" type="continuous">
-        <origin xyz="-${wheel_offset} ${wheel_separation/2} -${wheel_radius/2}" rpy="0 0 0"/>
+        <origin xyz="-${wheel_offset} ${wheel_separation/2} ${body_wheel_axle_offset}" rpy="0 0 0"/>
         <parent link="body_link"/>
         <child link="left_wheel_link"/>
@@ -180,5 +138,5 @@
     <!-- Right Wheel Joint -->
     <joint name="right_wheel_joint" type="continuous">
-        <origin xyz="-${wheel_offset} ${-wheel_separation/2} -${wheel_radius/2}" rpy="0 0 0"/>
+        <origin xyz="-${wheel_offset} ${-wheel_separation/2} ${body_wheel_axle_offset}" rpy="0 0 0"/>
         <parent link="body_link"/>
         <child link="right_wheel_link"/>
@@ -189,5 +147,5 @@
     <!-- Left Wheel2 Joint -->
     <joint name="left_wheel2_joint" type="continuous">
-        <origin xyz="${wheel_offset} ${wheel_separation/2} -${wheel_radius/2}" rpy="0 0 0"/>
+        <origin xyz="${wheel_offset} ${wheel_separation/2} ${body_wheel_axle_offset}" rpy="0 0 0"/>
         <parent link="body_link"/>
         <child link="left_wheel2_link"/>
@@ -198,5 +156,5 @@
     <!-- Right Wheel2 Joint -->
     <joint name="right_wheel2_joint" type="continuous">
-        <origin xyz="${wheel_offset} ${-wheel_separation/2} -${wheel_radius/2}" rpy="0 0 0"/>
+        <origin xyz="${wheel_offset} ${-wheel_separation/2} ${body_wheel_axle_offset}" rpy="0 0 0"/>
         <parent link="body_link"/>
         <child link="right_wheel2_link"/>
@@ -205,10 +163,34 @@
         <dynamics damping="0.1" friction="0.1"/>
     </joint>
-    <!-- Caster Wheel Joint (fixed) -->
-<!--    <joint name="caster_joint" type="fixed">
-        <origin xyz="${caster_offset} 0 -${caster_radius/2}" rpy="0 0 0"/>
-        <parent link="body_link"/>
-        <child link="caster_link"/>
-    </joint>-->
+    <!-- battery joint -->
+    <joint name="battery_joint" type="fixed">
+        <origin xyz=".007 0 ${body_battery_offset}" rpy="0 0 0"/>
+        <parent link="body_link"/>
+        <child link="battery_link"/>
+    </joint>
+    <!-- orin joint -->
+    <joint name="orin_joint" type="fixed">
+        <origin xyz=".010 0 ${battery_orin_offset}" rpy="0 0 0"/>
+        <parent link="battery_link"/>
+        <child link="orin_link"/>
+    </joint>
+    <!-- lidar joint -->
+    <joint name="lidar_joint" type="fixed">
+        <origin xyz="-.045 0 ${orin_lidar_offset}" rpy="0 0 0"/>
+        <parent link="orin_link"/>
+        <child link="lidar_link"/>
+    </joint>
+    <!-- camera joint -->
+    <joint name="d435_joint" type="fixed">
+        <origin xyz="${orin_d435_offset_x} 0 ${orin_d435_offset_z}" rpy="0 0 0"/>
+        <parent link="orin_link"/>
+        <child link="d435_link"/>
+    </joint>
+    <!-- gps joint -->
+    <joint name="gps_joint" type="fixed">
+        <origin xyz="${orin_gps_offset_x} ${orin_gps_offset_y} ${orin_gps_offset_z}" rpy="0 0 0"/>
+        <parent link="orin_link"/>
+        <child link="gps_link"/>
+    </joint>
     <!-- Gazebo Parameters -->
     <gazebo reference="body_link">
@@ -232,8 +214,4 @@
         <mu2>1.0</mu2>
     </gazebo>
-<!--    <gazebo reference="caster_link">
-        <mu1>0.000001</mu1>
-        <mu2>0.000001</mu2>
-    </gazebo>-->
     <!-- Gazebo Plugins -->
     <gazebo>
