Commit message: Update body_link -> base_link.

File: model/robot.xacro (robot description, xacro)
@@ -134,5 +134,5 @@
     <!-- Links -->
     <!-- Body Link -->
-    <xacro:box_link name="body_link" length="${body_length}" width="${body_width}" height="${body_height}" density="${body_density}" color="0.0 0.0 0.0 1.0"/>
+    <xacro:box_link name="base_link" length="${body_length}" width="${body_width}" height="${body_height}" density="${body_density}" color="0.0 0.0 0.0 1.0"/>
     <xacro:box_link name="battery_link" length="${battery_length}" width="${battery_width}" height="${battery_height}" density="${battery_density}" color="0.25 0.25 0.25 1.0"/>
     <xacro:box_link name="orin_link" length="${orin_length}" width="${orin_width}" height="${orin_height}" density="${orin_density}" color="0.45 0.45 0.45 1.0"/>
@@ -154,5 +154,5 @@
     <joint name="base_footprint_joint" type="fixed">
         <parent link="base_footprint"/>
-        <child link="body_link"/>
+        <child link="base_link"/>
         <origin xyz="0 0 ${body_ground_clearance + body_height/2.0}" rpy="0 0 0"/>
     </joint>
@@ -160,5 +160,5 @@
     <joint name="left_wheel_joint" type="continuous">
         <origin xyz="-${wheel_offset} ${wheel_separation/2} ${body_wheel_axle_offset}" rpy="0 0 0"/>
-        <parent link="body_link"/>
+        <parent link="base_link"/>
         <child link="left_wheel_link"/>
         <axis xyz="0 1 0"/>
@@ -169,5 +169,5 @@
     <joint name="right_wheel_joint" type="continuous">
         <origin xyz="-${wheel_offset} ${-wheel_separation/2} ${body_wheel_axle_offset}" rpy="0 0 0"/>
-        <parent link="body_link"/>
+        <parent link="base_link"/>
         <child link="right_wheel_link"/>
         <axis xyz="0 1 0"/>
@@ -178,5 +178,5 @@
     <joint name="left_wheel2_joint" type="continuous">
         <origin xyz="${wheel_offset} ${wheel_separation/2} ${body_wheel_axle_offset}" rpy="0 0 0"/>
-        <parent link="body_link"/>
+        <parent link="base_link"/>
         <child link="left_wheel2_link"/>
         <axis xyz="0 1 0"/>
@@ -187,5 +187,5 @@
     <joint name="right_wheel2_joint" type="continuous">
         <origin xyz="${wheel_offset} ${-wheel_separation/2} ${body_wheel_axle_offset}" rpy="0 0 0"/>
-        <parent link="body_link"/>
+        <parent link="base_link"/>
         <child link="right_wheel2_link"/>
         <axis xyz="0 1 0"/>
@@ -196,5 +196,5 @@
     <joint name="battery_joint" type="fixed">
         <origin xyz=".007 0 ${body_battery_offset}" rpy="0 0 0"/>
-        <parent link="body_link"/>
+        <parent link="base_link"/>
         <child link="battery_link"/>
     </joint>
@@ -225,5 +225,5 @@
     <!-- Gazebo Parameters -->
     <!--
-    <gazebo reference="body_link">
+    <gazebo reference="base_link">
         <mu1>1.0</mu1>
         <mu2>0.5</mu2>
@@ -269,4 +269,5 @@
             <topic>cmd_vel</topic>
             <odom_topic>odom</odom_topic>
+            <frame_id>odom</frame_id>
             <child_frame_id>base_footprint</child_frame_id>
             <tf_topic>/tf</tf_topic>
@@ -375,5 +376,5 @@
       </sensor>
     </gazebo>
-    <gazebo reference="body_link">
+    <gazebo reference="base_link">
       <sensor name='ugv_imu' type='imu'>
         <always_on>true</always_on>

File: model/robot_third_person.xacro (robot description, xacro)
@@ -134,5 +134,5 @@
     <!-- Links -->
     <!-- Body Link -->
-    <xacro:box_link name="body_link" length="${body_length}" width="${body_width}" height="${body_height}" density="${body_density}" color="0.0 0.0 0.0 1.0"/>
+    <xacro:box_link name="base_link" length="${body_length}" width="${body_width}" height="${body_height}" density="${body_density}" color="0.0 0.0 0.0 1.0"/>
     <xacro:box_link name="battery_link" length="${battery_length}" width="${battery_width}" height="${battery_height}" density="${battery_density}" color="0.25 0.25 0.25 1.0"/>
     <xacro:box_link name="orin_link" length="${orin_length}" width="${orin_width}" height="${orin_height}" density="${orin_density}" color="0.45 0.45 0.45 1.0"/>
@@ -154,5 +154,5 @@
     <joint name="base_footprint_joint" type="fixed">
         <parent link="base_footprint"/>
-        <child link="body_link"/>
+        <child link="base_link"/>
         <origin xyz="0 0 ${body_ground_clearance + body_height/2.0}" rpy="0 0 0"/>
     </joint>
@@ -160,5 +160,5 @@
     <joint name="left_wheel_joint" type="continuous">
         <origin xyz="-${wheel_offset} ${wheel_separation/2} ${body_wheel_axle_offset}" rpy="0 0 0"/>
-        <parent link="body_link"/>
+        <parent link="base_link"/>
         <child link="left_wheel_link"/>
         <axis xyz="0 1 0"/>
@@ -169,5 +169,5 @@
     <joint name="right_wheel_joint" type="continuous">
         <origin xyz="-${wheel_offset} ${-wheel_separation/2} ${body_wheel_axle_offset}" rpy="0 0 0"/>
-        <parent link="body_link"/>
+        <parent link="base_link"/>
         <child link="right_wheel_link"/>
         <axis xyz="0 1 0"/>
@@ -178,5 +178,5 @@
     <joint name="left_wheel2_joint" type="continuous">
         <origin xyz="${wheel_offset} ${wheel_separation/2} ${body_wheel_axle_offset}" rpy="0 0 0"/>
-        <parent link="body_link"/>
+        <parent link="base_link"/>
         <child link="left_wheel2_link"/>
         <axis xyz="0 1 0"/>
@@ -187,5 +187,5 @@
     <joint name="right_wheel2_joint" type="continuous">
         <origin xyz="${wheel_offset} ${-wheel_separation/2} ${body_wheel_axle_offset}" rpy="0 0 0"/>
-        <parent link="body_link"/>
+        <parent link="base_link"/>
         <child link="right_wheel2_link"/>
         <axis xyz="0 1 0"/>
@@ -196,5 +196,5 @@
     <joint name="battery_joint" type="fixed">
         <origin xyz=".007 0 ${body_battery_offset}" rpy="0 0 0"/>
-        <parent link="body_link"/>
+        <parent link="base_link"/>
         <child link="battery_link"/>
     </joint>
@@ -225,5 +225,5 @@
     <!-- Gazebo Parameters -->
     <!--
-    <gazebo reference="body_link">
+    <gazebo reference="base_link">
         <mu1>1.0</mu1>
         <mu2>0.5</mu2>
@@ -375,5 +375,5 @@
       </sensor>
     </gazebo>
-    <gazebo reference="body_link">
+    <gazebo reference="base_link">
       <sensor name='ugv_imu' type='imu'>
         <always_on>true</always_on>
