Commit message: Simulation updates after a round of updates and debugging.

File: model/ugv.xacro (robot description, xacro)
@@ -151,4 +151,5 @@
         </inertial>
     </link>
+    <link name="camera_optical_link"/>
     <!-- Joints -->
     <joint name="base_footprint_joint" type="fixed">
@@ -216,4 +217,10 @@
         <parent link="orin_link"/>
         <child link="camera_link"/>
+    </joint>
+    <!-- optical frame ${-3.1415927/2} 0 ${-3.1415927/2} -->
+    <joint name="camera_optical_joint" type="fixed">
+        <origin xyz="0 0 0" rpy="0 0 0"/>
+        <parent link="camera_link"/>
+        <child link="camera_optical_link"/>
     </joint>
     <!-- gps joint -->
@@ -288,12 +295,12 @@
     <!-- Gazebo sensors -->
     <gazebo reference="camera_link">
-      <sensor name="d435_depth" type="depth_camera">
-        <pose>0 0 0 0 -0 0</pose>
+      <sensor name="color_camera" type="rgbd_camera">
+        <pose>0.0 0.0 0 0 0 0</pose>
         <always_on>true</always_on>
         <visualize>true</visualize>
         <update_rate>30</update_rate>
-        <topic>/d435_depth_camera/image_raw</topic>
+        <topic>/camera</topic>
+        <gz_frame_id>camera_optical_link</gz_frame_id>
         <camera name="intel_realsense_r200">
-          <camera_info_topic>depth_camera/camera_info</camera_info_topic>
           <horizontal_fov>1.02974</horizontal_fov>
           <image>
@@ -303,5 +310,5 @@
           </image>
           <clip>
-            <near>0.01</near>
+            <near>0.05</near>
             <far>200</far>
           </clip>
@@ -317,27 +324,26 @@
       </sensor>
     </gazebo>
+    <xacro:if value='false'>
     <gazebo reference="camera_link">
-      <sensor name="d435_rgb_camera" type="camera">
-        <pose>0 0 0 0 -0 0</pose>
+      <sensor name="depth_camera" type="depth_camera">
+        <pose>0 0 0 0 0 0</pose>
         <always_on>true</always_on>
         <visualize>true</visualize>
         <update_rate>30</update_rate>
-        <topic>/d435_rgb_camera/image_raw</topic>
+        <topic>/camera/depth/image_raw</topic>
+        <gz_frame_id>camera_optical_link</gz_frame_id>
         <camera name="intel_realsense_r200">
           <horizontal_fov>1.02974</horizontal_fov>
           <image>
-            <width>640</width>
-            <height>480</height>
+            <width>424</width>
+            <height>240</height>
             <format>R8G8B8</format>
           </image>
           <clip>
-            <near>0.01</near>
+            <near>0.05</near>
             <far>200</far>
           </clip>
           <noise>
             <type>gaussian</type>
-            <!-- Noise is sampled independently per pixel on each frame.
-                  That pixel's noise value is added to each of its color
-                  channels, which at that point lie in the range [0,1]. -->
             <mean>0.0</mean>
             <stddev>0.007</stddev>
@@ -346,4 +352,5 @@
       </sensor>
     </gazebo>
+    </xacro:if>
     <gazebo reference="lidar_link">
       <sensor name='hls_lfcd_lds' type='gpu_lidar'>
@@ -381,4 +388,5 @@
         <update_rate>20</update_rate>
         <topic>imu</topic>
+        <gz_frame_id>base_link</gz_frame_id>
         <imu>
           <angular_velocity>

Commit message: Add calibratable ugv.xacro file to gazebo package. This ugv.xacro mirrors the ugv.xacro for the real robot - with the calibration joint set to 0 for all parameters (unit transform).

File: model/ugv.xacro (robot description, xacro)
@@ -138,5 +138,5 @@
     <xacro:box_link name="orin_link" length="${orin_length}" width="${orin_width}" height="${orin_height}" density="${orin_density}" color="0.45 0.45 0.45 1.0"/>
     <xacro:box_link name="lidar_link" length="${lidar_length}" width="${lidar_width}" height="${lidar_height}" density="${lidar_density}" color="0.0 0.0 0.0 1.0"/>
-    <xacro:box_link name="camera_link" length="${d435_length}" width="${d435_width}" height="${d435_height}" density="${d435_density}" color="0.7 0.7 0.7 1.0"/>
+    <xacro:box_link name="camera_pre_link" length="${d435_length}" width="${d435_width}" height="${d435_height}" density="${d435_density}" color="0.7 0.7 0.7 1.0"/>
     <xacro:box_link name="gps_link" length="${gps_length}" width="${gps_width}" height="${gps_height}" density="${gps_density}" color="1.0 1.0 1.0 1.0"/>
     <xacro:wheel_link name="left_wheel_link" radius="${wheel_radius}" width="${wheel_width}" density="${wheel_density}" color="0.1 0.1 0.1 1.0"/>
@@ -152,4 +152,5 @@
     </link>
     <link name="camera_optical_link"/>
+    <link name="camera_link"/>
     <!-- Joints -->
     <joint name="base_footprint_joint" type="fixed">
@@ -216,4 +217,10 @@
 	    <origin xyz="${orin_d435_offset_x} 0 ${orin_d435_offset_z-.02}" rpy="0 ${35.0*3.1416/180.0} 0"/>
         <parent link="orin_link"/>
+        <child link="camera_pre_link"/>
+    </joint>
+    <!-- camera calibration joint -->
+    <joint name="d435_calibration_joint" type="fixed">
+	    <origin xyz="0 0 0" rpy="0 0 0"/>
+        <parent link="camera_pre_link"/>
         <child link="camera_link"/>
     </joint>
